Commit message: feat: change in bot, script, and movement node

File: ws/install/box_bot_description/share/box_bot_description/urdf/box_bot.urdf (robot description, URDF)
Before this commit: robot box_bot, 15 links, 14 joints
Links:
- removed link pointcloud_link
- removed link rgb_camera_link_frame
- link chassis: geometry collision cylinder length=0.1 radius=0.05; visual cylinder length=0.1 radius=0.05
Joints:
- removed joint pointcloud_link_joint
- removed joint rgb_camera_link_frame_joint

Commit message: checkpoint

File: ws/install/box_bot_description/share/box_bot_description/urdf/box_bot.urdf (robot description, URDF)
Before this commit: robot box_bot, 13 links, 12 joints
Links:
- link back_pitch_link: mass 0.001 -> 0.005
- link front_pitch_link: mass 0.001 -> 0.005

Commit message: feat: now the bot can stop

File: ws/install/box_bot_description/share/box_bot_description/urdf/box_bot.urdf (robot description, URDF)
Before this commit: robot box_bot, 13 links, 12 joints
Links:
- link back_pitch_link: mass 0.005 -> 0.001
- link chassis: geometry collision cylinder length=0.1 radius=0.1; visual cylinder length=0.1 radius=0.1
- link front_pitch_link: mass 0.005 -> 0.001
Joints:
- joint back_yaw_joint: origin xyz=-0.04 0 -0.05 rpy=0 0 0 -> xyz=-0.08 0 -0.05 rpy=0 0 0
- joint front_yaw_joint: origin xyz=0.04 0 -0.05 rpy=0 0 0 -> xyz=0.08 0 -0.05 rpy=0 0 0
- joint joint_left_wheel: origin xyz=0 -0.05 -0.025 rpy=0 0 0 -> xyz=0 -0.1 -0.025 rpy=0 0 0
- joint joint_right_wheel: origin xyz=0 0.05 -0.025 rpy=0 0 0 -> xyz=0 0.1 -0.025 rpy=0 0 0
- joint laser_scan_link_joint: origin xyz=0.0 0.0 0.05 rpy=0 0 0 -> xyz=0.0 0.0 0.09 rpy=0 0 0
