Commit message: refactor:change pkg names

File: ws/src/robot_description/urdf/reactive_robot.urdf (robot description, URDF)
Before this commit: robot reactive_robot, 15 links, 14 joints
Links:
- removed link pointcloud_link
- removed link rgb_camera_link_frame
- link chassis: geometry collision cylinder length=0.1 radius=0.1; visual cylinder length=0.1 radius=0.1
Joints:
- removed joint pointcloud_link_joint
- removed joint rgb_camera_link_frame_joint
- joint back_yaw_joint: origin xyz=-0.04 0 -0.05 rpy=0 0 0 -> xyz=-0.08 0 -0.05 rpy=0 0 0
- joint front_yaw_joint: origin xyz=0.04 0 -0.05 rpy=0 0 0 -> xyz=0.08 0 -0.05 rpy=0 0 0
- joint joint_left_wheel: origin xyz=0 -0.05 -0.025 rpy=0 0 0 -> xyz=0 -0.1 -0.025 rpy=0 0 0
- joint joint_right_wheel: origin xyz=0 0.05 -0.025 rpy=0 0 0 -> xyz=0 0.1 -0.025 rpy=0 0 0
- joint laser_scan_link_joint: origin xyz=0.0 0.0 0.05 rpy=0 0 0 -> xyz=0.0 0.0 0.09 rpy=0 0 0
